File: HW/USB_Midi_Pots/main.brd (EAGLE design)
At the start: 86.3 x 86.7 mm, 61 parts, among them SW1 EC12E_SW

Commit message: HW update
Parts:
- added C20: (no value), Ai_Passives:CAP-0805
- added USB2: (no value), pinhead:1X04
- moved C5 4.96 mm to (44.5, 85.7), turned to 270 degrees
- moved C18 2.54 mm to (55.2, 87.6)
- moved C16 2.54 mm to (84.5, 87.6)
- moved C15 1.27 mm to (99.1, 87.6)
- moved C17 0.63 mm to (69.2, 87.6)
Connections:
- net +5V: now also C20.1, USB2.4
- net GND: now also C20.2, USB2.1
- net N$1: now also USB2.3
- net N$2: now also USB2.2
Routing:
- net +5V: track 230.0 -> 264.1 mm, vias 5 -> 7
- net FADER3: track 38.9 -> 54.7 mm
- net FADER2: track 28.3 -> 41.1 mm
- net FADER4: track 56.4 -> 68.7 mm
- net GND: track 0.00 -> 2.31 mm, vias 524 -> 506
- net N$1: track 16.5 -> 18.1 mm, vias 1 -> 0
- net FADER1: track 52.4 -> 53.3 mm
- net N$2: track 19.0 -> 18.8 mm, vias 1 -> 0
Other:
- board text added: "o"

Commit message: Board Update
Parts:
- added D7: (no value), Ai_LED:LED-0603
- added L3: (no value), Ai_Passives:IND-0603
- added R6: (no value), Ai_Passives:RES-0603
- moved C5 30.3 mm to (19.1, 69.2)
- moved C20 28.4 mm to (64.8, 80.6)
- moved C3 28.4 mm to (55.0, 29.5)
- moved JP6 28.4 mm to (57.8, 5.08)
- moved JP8 28.4 mm to (72.4, 5.08)
- moved R10 28.4 mm to (12.1, 38.7)
- moved U$1 28.4 mm to (46.9, 43.1)
- moved JP2 28.4 mm to (28.6, 5.08)
- moved R1 28.4 mm to (10.2, 67.9)
- moved R13 28.4 mm to (14.6, 31.1)
- moved R9 28.4 mm to (12.7, 36.8)
- moved C10 28.4 mm to (49.5, 34.0)
- moved C13 28.4 mm to (51.2, 52.8)
- moved C15 28.4 mm to (73.7, 74.9)
- moved C17 28.4 mm to (43.8, 74.9)
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Connections:
- new net N$36: R6.1, U$1.1
- new net N$38: D7.A, R6.2
- new net N$40: L3.1, U$2.1, USB2.4
- net +5V: now also L3.2; no longer U$2.1, USB2.4
- net GND: now also D7.C
Routing:
- net N$25: track 25.3 -> 61.7 mm, vias 0 -> 1
- net N$8: track 23.5 -> 58.7 mm, vias 0 -> 1
- net N$36: track 0.00 -> 35.0 mm, vias 0 -> 1
- net N$40: track 0.00 -> 8.73 mm
- net +5V: track 264.1 -> 260.8 mm, vias 7 -> 5
- net N$38: track 0.00 -> 2.80 mm
- net N$14: track 4.81 -> 5.31 mm
- net GND: vias 506 -> 465

Commit message: Rotary Encoder Test and other Board Layouts
Parts:
- C4: value 1uF -> 4.7uF
- C7: value (none) -> 1uF
